File: Blance_Car.kicad_pcb (KiCad board)
At the start: 2 copper layers, 60 x 100 mm, 22 parts, among them J1 XT60PW-M, J2 Conn_01x02_Female, J3 Conn_01x02_Female, U1 ras_head, U2 L298HN, U3 KA78M05_TO252

Commit message: 2nd
Parts:
- moved h3 5.08 mm to (27.9, 49.5)
- moved h2 3.81 mm to (73.7, 50.8)
- moved C5 2.84 mm to (69.8, 64.8), turned to 180 degrees
Routing:
- net /Motor_sensor_8: track 17.5 -> 12.4 mm
- net /Motor_sensor_7: track 21.0 -> 16.0 mm
- net /Motor_sensor_6: track 24.6 -> 19.6 mm
- net /Motor_sensor_5: track 28.2 -> 23.2 mm
- net /SDA: track 51.2 -> 46.9 mm
- net /Motor_sensor_4: track 34.9 -> 31.1 mm
- net /Motor_sensor_3: track 31.3 -> 27.5 mm
- net /Motor_sensor_2: track 27.7 -> 23.9 mm
- net /Motor_sensor_1: track 24.1 -> 20.3 mm
- net GND: track 37.4 -> 40.0 mm
- net +5V: track 53.5 -> 52.3 mm
- net /GPIO13(PWM1): track 66.1 -> 65.0 mm
